File: Interface.kicad_sch (KiCad schematic)
At the start: 11 parts, among them J1 Power, J2 Digital/PWM, J3 Analog, J4 Digital/PWM, J6 CX90M

Commit message: update: 更新PCB
Parts:
- added D4: BLUE, LED_SMD:LED_0603_1608Metric, symbol Device:LED
- added R27: 10k, Resistor_SMD:R_0402_1005Metric, symbol Device:R
- added U11: 0524P, Package_SON:USON-10_2.5x1.0mm_P0.5mm, symbol Power_Protection:TPD4EUSB30
Connections:
- net +3V3: no longer R21.2, R22.2
- net D13: now also R27.1
- net GND: now also D4.1 (K), U11.3 (GND), U11.4 (D2+), U11.5 (D2-), U11.6 (NC), U11.7 (NC), U11.8 (GND)
- net USB_D+: now also U11.2 (D1-), U11.9 (NC)
- net USB_D-: now also U11.1 (D1+), U11.10 (NC)
- new net: D4.2 (A), R27.2
- new net VDD33_1: R21.2, R22.2
