File: Audio.kicad_sch (KiCad schematic)
At the start: 19 parts, among them U6 NS4150B

Commit message: update: 更新PCB
Parts:
- added R26: 0R, Resistor_SMD:R_0603_1608Metric, symbol Device:R
Connections:
- net GND: now also R26.1; no longer C32.2, C33.2, C34.2, C35.2, C40.1, C41.2, C45.2, MIC1.2 (GND), MIC1.3 (GND), R12.2, U6.7 (GND)
- new net GNDA: C32.2, C33.2, C34.2, C35.2, C40.1, C41.2, C45.2, MIC1.2 (GND), MIC1.3 (GND), R12.2, R26.2, U6.7 (GND)

Commit message: update:
Changed lines of the file:
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@@
-	)
-	(junction
-		(at 62.23 31.75)
-		(diameter 0)
-		(color 0 0 0 0)
 	)
 	(junction
@@
 	)
 	(junction
+		(at 62.23 30.48)
+		(diameter 0)
+		(color 0 0 0 0)
+	)
+	(junction
 		(at 90.17 30.48)
 		(diameter 0)
@@
 	(wire
 		(pts
-			(xy 62.23 33.02) (xy 62.23 31.75)
+			(xy 62.23 30.48) (xy 62.23 33.02)
 		)
 		(stroke
@@
 	(wire
 		(pts
-			(xy 62.23 27.94) (xy 62.23 31.75)
+			(xy 62.23 27.94) (xy 62.23 30.48)
 		)
 		(stroke
@@
 	(wire
 		(pts
-			(xy 62.23 31.75) (xy 66.04 31.75)
+			(xy 62.23 30.48) (xy 66.04 30.48)
 		)
 		(stroke
@@
 		)
 	)
-	(label "PA_EN"
-		(at 66.04 31.75 0)
+	(hierarchical_label "PA_EN"
+		(shape input)
+		(at 66.04 30.48 0)
 		(fields_autoplaced yes)
 		(effects
@@
 				(size 1.27 1.27)
 			)
-			(justify left bottom)
-		)
-	)
+			(justify left)
+		)
+	)
