File: SFduino-UNO-S2.kicad_pcb (KiCad board)
At the start: 2 copper layers, 68.6 x 53.3 mm, 116 parts, among them J1 Power, J2 Digital/PWM, J3 Analog, J4 Digital/PWM, J5 FPC 16p 0.5mm, J6 CX90M, J7 MX1.25 2P, Q1 SI2305, Q2 SI2305, SW1 SKHMQLE010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

Commit message: update: 更新PCB
Parts:
- added C56: 10u, Capacitor_SMD:C_0402_1005Metric, F.Cu at (113.4, 64.8)
- added C57: 1u, Capacitor_SMD:C_0402_1005Metric, F.Cu at (123.2, 62.4)
- added C58: 0.1u, Capacitor_SMD:C_0402_1005Metric, F.Cu at (144.9, 73.2)
- added C59: 0.1u, Capacitor_SMD:C_0402_1005Metric, F.Cu at (124.9, 60.1)
- added D4: BLUE, LED_SMD:LED_0603_1608Metric, F.Cu at (142.4, 56.8)
- added Q3: AO3407, Package_TO_SOT_SMD:SOT-23, F.Cu at (116.6, 56.4)
- added R23: 100k, Resistor_SMD:R_0402_1005Metric, F.Cu at (118.8, 57.4)
- added R24: 100R, Resistor_SMD:R_0402_1005Metric, F.Cu at (124.9, 62.9)
- added R25: 100R, Resistor_SMD:R_0402_1005Metric, F.Cu at (125.8, 62.9)
- added R26: 0R, Resistor_SMD:R_0603_1608Metric, F.Cu at (133.4, 80.2)
- added R27: 10k, Resistor_SMD:R_0402_1005Metric, F.Cu at (142.4, 59.8)
- added U11: 0524P, Package_SON:USON-10_2.5x1.0mm_P0.5mm, F.Cu at (108.3, 61.6)
- C50, C52: value 1u -> 0.1u
- Y2: footprint Crystal:Crystal_SMD_2016-4Pin_2.0x1.6mm -> Crystal:Crystal_SMD_2520-4Pin_2.5x2.0mm
- moved Q1 128.9 mm to (116.3, 65.9), turned to 90 degrees
- moved D1 127.0 mm to (111.8, 67.2), turned to 180 degrees
- moved U3 122.6 mm to (111.8, 56.4), turned to 180 degrees
- moved C40 121.8 mm to (120.1, 76.6), turned to -90 degrees
- moved C37 119.8 mm to (119.2, 77.5), turned to 90 degrees
- moved C38 119.0 mm to (125.4, 95.0), turned to 90 degrees
- moved C35 119.0 mm to (120.1, 78.4), turned to -90 degrees
- moved C41 118.8 mm to (124.5, 95.0), turned to 90 degrees
- moved C22 118.8 mm to (120.0, 56.4), turned to -90 degrees
- moved FB1 118.8 mm to (121.5, 77.9), turned to 180 degrees
- moved C18 118.6 mm to (109.2, 56.4), turned to 90 degrees
- moved FB2 118.4 mm to (121.5, 77.0), turned to 180 degrees
- moved R20 118.2 mm to (110.6, 64.8), turned to 90 degrees
- moved C21 117.7 mm to (121.5, 56.4), turned to -90 degrees
- moved C34 117.6 mm to (123.5, 95.0), turned to 90 degrees
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Connections:
- C19 pad 1: +5V -> Net-(Q3-D)
- C32 pad 2: GND -> GNDA
- C33 pad 2: GND -> GNDA
- C34 pad 2: GND -> GNDA
- C35 pad 2: GND -> GNDA
- C40 pad 1: GND -> GNDA
- C41 pad 2: GND -> GNDA
- C45 pad 2: GND -> GNDA
- C49 pad 1: +3V3 -> VBUS
- C50 pad 1: +3V3 -> Net-(U8-VDD33)
- C51 pad 1: +3V3 -> Net-(U9-V3)
- C52 pad 1: +3V3 -> Net-(U9-V3)
- J2 pad 1: /I2C_SCL -> /PA22
- J2 pad 10: /PA23 -> /PA10
- J2 pad 2: /I2C_SDA -> /PA23
- J2 pad 8: /PA44 -> /PA11
- J2 pad 9: /PA38 -> /PA20
- J3 pad 1: /PA34 -> /PA29
- J3 pad 2: /PA33 -> /PA30
- J3 pad 3: /PA32 -> /PA31
- J3 pad 4: /PA31 -> /PA32
- J3 pad 5: /PA30 -> /PA33
- J3 pad 6: /PA29 -> /PA34
- J4 pad 1: /PA22 -> /PA9
- J4 pad 2: /PA20 -> /PA26
- J4 pad 3: /PA11 -> /PA27
- J4 pad 4: /PA10 -> /PA1
- J4 pad 5: /PA9 -> /PA38
- J4 pad 6: /PA1 -> /PA44
- J5 pad 1: +5V -> GND
- J5 pad 10: /DISPLAY_D8 -> /DISPLAY_D5
- J5 pad 11: /DISPLAY_D9 -> /DISPLAY_D4
- J5 pad 12: /DISPLAY_D10 -> /DISPLAY_D3
- J5 pad 13: /DISPLAY_D11 -> /DISPLAY_D2
- J5 pad 14: /DISPLAY_D12 -> /DISPLAY_D1
- J5 pad 15: /DISPLAY_D13 -> /DISPLAY_D0
- J5 pad 16: GND -> +5V
- J5 pad 2: /DISPLAY_D0 -> /DISPLAY_D13
- J5 pad 3: /DISPLAY_D1 -> /DISPLAY_D12
- J5 pad 4: /DISPLAY_D2 -> /DISPLAY_D11
- J5 pad 5: /DISPLAY_D3 -> /DISPLAY_D10
- J5 pad 6: /DISPLAY_D4 -> /DISPLAY_D9
- J5 pad 7: /DISPLAY_D5 -> /DISPLAY_D8
- J5 pad 8: /DISPLAY_D6 -> /DISPLAY_D7
- J5 pad 9: /DISPLAY_D7 -> /DISPLAY_D6
- MIC1 pad 2: GND -> GNDA
- MIC1 pad 3: GND -> GNDA
- R12 pad 2: GND -> GNDA
- R21 pad 1: /I2C_SCL -> /PA22
- R21 pad 2: +3V3 -> VDD33_1
- R22 pad 1: /I2C_SDA -> /PA23
- R22 pad 2: +3V3 -> VDD33_1
- U1 pad 6: /I2C_SDA -> /PA27
- U1 pad 7: /I2C_SCL -> /PA26
- U3 pad 1: +5V -> Net-(Q3-D)
- U6 pad 7: GND -> GNDA
- U8 pad 10: /UART_D+ -> /SF_D+
- U8 pad 15: +3V3 -> VBUS
- U8 pad 16: +3V3 -> Net-(U8-VDD33)
- U8 pad 5: unconnected-(U8-DM3-Pad5) -> /UART_D-
- U8 pad 6: unconnected-(U8-DP3-Pad6) -> /UART_D+
- U8 pad 7: /SF_D- -> unconnected-(U8-DM2-Pad7)
- U8 pad 8: /SF_D+ -> unconnected-(U8-DP2-Pad8)
- U8 pad 9: /UART_D- -> /SF_D-
- U9 pad 1: +3V3 -> Net-(U9-V3)
- U9 pad 3: +3V3 -> VBUS
- U9 pad 4: /PA18 -> Net-(U9-TXD)
- U9 pad 5: /PA19 -> Net-(U9-RXD)
- U9 pad 6: +3V3 -> Net-(U9-V3)
Routing:
- net VBAT: track 0.00 -> 91.0 mm, vias 0 -> 6
- net /SF_D-: track 0.00 -> 72.4 mm, vias 0 -> 2
- net /SF_D+: track 0.00 -> 71.7 mm, vias 0 -> 2
- net VIN: track 0.00 -> 54.3 mm, vias 0 -> 2
- net /MIC_BIAS: track 0.00 -> 50.3 mm, vias 0 -> 2
- net /PA18: track 0.00 -> 50.0 mm, vias 0 -> 2
- net /PA22: track 0.00 -> 46.7 mm
- net /PA19: track 0.00 -> 45.3 mm, vias 0 -> 2
- net /PA23: track 0.00 -> 44.2 mm
- net /PA29: track 0.00 -> 42.1 mm, vias 0 -> 1
- net /MIC_IN: track 0.00 -> 41.9 mm, vias 0 -> 2
- net /PA30: track 0.00 -> 40.0 mm, vias 0 -> 1
- net /PA11: track 0.00 -> 39.6 mm, vias 0 -> 2
- net /PA10: track 0.00 -> 38.1 mm, vias 0 -> 2
- net +5V: track 0.00 -> 37.6 mm, vias 0 -> 2
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- added copper zone on B.Cu, net GNDA
- added copper zone on F.Cu, net GNDA
Other:
- board text removed: "ICSP"

Commit message: update:
Parts:
- moved C33 6.86 mm to (123.7, 73.8), turned to 0 degrees
- moved C32 5.18 mm to (124.3, 75.0), turned to 0 degrees
Connections:
- R10 pad 1: /PA1 -> /PA10
- U5 pad 3: /PA1 -> /PA10
- U7 pad 4: /PA1 -> /PA10
Routing:
- net +5V: track 37.6 -> 110.5 mm, vias 2 -> 9
- net VBUS: track 3.51 -> 64.5 mm, vias 0 -> 6
- net /PA18: track 50.0 -> 81.4 mm, vias 2 -> 3
- net /PA19: track 45.3 -> 74.0 mm, vias 2 -> 3
- net /PA10: track 38.1 -> 62.8 mm, vias 2 -> 4
- net Net-(U9-V3): track 0.00 -> 10.4 mm, vias 0 -> 2
- net GND: track 28.0 -> 20.4 mm, vias 16 -> 20
- net Net-(U9-RXD): track 0.00 -> 5.84 mm
- net Net-(U9-TXD): track 0.00 -> 3.88 mm
- net /EN: track 0.00 -> 2.77 mm
- net Net-(U9-DTR): track 0.00 -> 2.54 mm
- net Net-(Q2-D): track 25.1 -> 27.6 mm
- net Net-(U8-VDD33): track 0.00 -> 2.23 mm
- net VIN: track 54.3 -> 55.3 mm, vias 2 -> 4
- net /PA32: track 37.0 -> 37.9 mm
Other:
- outline, holes or cut-outs redrawn

Commit message: update:
Parts:
- added C60: TBD, Capacitor_SMD:C_0402_1005Metric, F.Cu at (158.1, 66.9)
- added C61: TBD, Capacitor_SMD:C_0402_1005Metric, F.Cu at (161.1, 67.8)
- added C62: 0.1u, Capacitor_SMD:C_0402_1005Metric, F.Cu at (156.7, 66.9)
- added SW2: SK-3293S, My Switch:SW-SMD_SK-3293S_mini_7P, F.Cu at (162.6, 58.4)
- added U12: FM8625H, Package_LGA:Infineon_PG-TSNP-6-10_0.7x1.1mm_0.7x1.1mm_P0.4mm, F.Cu at (157.9, 70.2)
- R2: value 0R -> TBD_R
- R3: value 0R -> 1k
- moved R3 9.71 mm to (159.2, 58.4), turned to 180 degrees
- moved U2 5.46 mm to (141.7, 82.2)
- moved C15 5.46 mm to (137.7, 80.8), turned to -135 degrees
- moved C9 5.46 mm to (141.3, 70.7)
- moved C8 5.46 mm to (140.6, 71.3)
- moved R21 5.46 mm to (143.1, 69.2)
- moved C13 5.46 mm to (141.9, 70.0)
- moved C5 5.46 mm to (140.0, 72.0)
- moved R22 5.46 mm to (143.8, 68.5)
- moved C2 5.46 mm to (140.9, 75.8)
- moved C58 5.46 mm to (139.6, 74.5)
- moved C6 5.46 mm to (142.8, 77.7)
- moved C10 5.46 mm to (140.6, 69.4)
- moved C1 5.46 mm to (141.5, 76.4)
- moved L1 5.46 mm to (138.7, 73.2)
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Connections:
- C16 pad 1: Net-(C16-Pad1) -> /RF2
- C17 pad 1: Net-(U1B-ANT) -> Net-(AE1-A)
- R1 pad 1: Net-(U1B-ANT) -> /RF2
- R1 pad 2: Net-(C16-Pad1) -> Net-(AE1-A)
- R12 pad 1: /Audio/PA_EN -> /PA9
- R2 pad 1: Net-(AE1-A) -> /RF1
- R2 pad 2: Net-(C16-Pad1) -> Net-(AE2-A)
- R3 pad 1: Net-(C16-Pad1) -> Net-(SW2-B)
- R3 pad 2: Net-(AE2-A) -> /RF_CTRL
- U1 pad 53: Net-(U1B-ANT) -> Net-(U12-RFIN)
- U6 pad 1: /Audio/PA_EN -> /PA9
Routing:
- net /EN: track 2.77 -> 72.7 mm, vias 0 -> 2
- net VDD33_1: track 5.21 -> 69.5 mm, vias 1 -> 6
- net VIN: track 55.3 -> 108.6 mm, vias 4 -> 2
- net +3V3: track 0.00 -> 45.9 mm, vias 0 -> 1
- net GND: track 20.4 -> 60.5 mm, vias 20 -> 84
- net /PA9: track 35.4 -> 69.8 mm, vias 2 -> 3
- net +5V: track 110.5 -> 143.8 mm, vias 9 -> 8
- net VCC: track 6.76 -> 30.5 mm, vias 0 -> 2
- net VSYS: track 5.49 -> 22.4 mm, vias 0 -> 2
- net /RF_CTRL: track 0.00 -> 14.2 mm, vias 0 -> 2
- net /PA18: track 81.4 -> 68.5 mm
- net /SF_D-: track 72.4 -> 60.3 mm
- net /SF_D+: track 71.7 -> 59.8 mm
- net /PA29: track 42.1 -> 33.3 mm
- net /PA19: track 74.0 -> 65.4 mm
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- added copper zone on B.Cu, net GND
- added copper zone on F.Cu, net GND
- added copper zone on In1.Cu, net GND
Other:
- copper layers 2 -> 4
- board text added: "+3V3"
- board text added: "+5V"
- board text added: "ANT"
- board text added: "D13"
- board text added: "EN"
- board text added: "GND"
- board text added: "IPEX"
- board text added: "NC"
- board text added: "PA1"
- board text added: "PA10"
- board text added: "PA11"
- board text added: "PA18"
- board text added: "PA19"
- board text added: "PA20"
- board text added: "PA22"
- board text added: "PA23"
- board text added: "PA24"
- board text added: "PA25"
- board text added: "PA26"
- board text added: "PA27"
- board text added: "PA28"
- board text added: "PA29"
- board text added: "PA30"
- board text added: "PA31"
- board text added: "PA32"
- board text added: "PA33"
- board text added: "PA34"
- board text added: "PA38"
- board text added: "PA44"
- board text added: "PA9"
- board text added: "RESET"
- board text added: "VIN"
