File: SFduino-UNO-S2.kicad_sch (KiCad schematic)
At the start: 27 parts, among them J5 FPC 16p 0.5mm, SW1 SKHMQLE010, U1 SF32LB527UD6, U2 PY25Q128HA-WXH-IR, U8 CH334P, U9 CH343P, Y1 48M, Y2 12M

Commit message: fix: 修复电源架构
Parts:
- added C56: 10u, Capacitor_SMD:C_0402_1005Metric, symbol Device:C
- added C57: 1u, Capacitor_SMD:C_0402_1005Metric, symbol Device:C
- C50, C52: value 1u -> 0.1u
Connections:
- net GND: now also C56.2, C57.2
- net VBUS: now also C49.1, U8.15 (V5), U9.3 (VDD5), C57.1
- removed net +3V3: C49.1, C50.1, C51.1, C52.1, U8.15 (V5), U8.16 (VDD33), U9.1 (VIO), U9.3 (VDD5), U9.6 (V3)
- new net: C51.1, C52.1, U9.1 (VIO), U9.6 (V3)
- new net: C50.1, C56.1, U8.16 (VDD33)
Other:
- moved on the sheet: C50, C52

Commit message: update: 更新PCB
Parts:
- added R24, R25: 100R, Resistor_SMD:R_0402_1005Metric, symbol Device:R
- Y2: footprint Crystal:Crystal_SMD_2016-4Pin_2.0x1.6mm -> Crystal:Crystal_SMD_2520-4Pin_2.5x2.0mm
Connections:
- net +5V: now also J5.16 (Pin_16); no longer J5.1 (Pin_1)
- net DISPLAY_D0: now also J5.15 (Pin_15); no longer J5.2 (Pin_2)
- net DISPLAY_D1: now also J5.14 (Pin_14); no longer J5.3 (Pin_3)
- net DISPLAY_D10: now also J5.5 (Pin_5); no longer J5.12 (Pin_12)
- net DISPLAY_D11: now also J5.4 (Pin_4); no longer J5.13 (Pin_13)
- net DISPLAY_D12: now also J5.3 (Pin_3); no longer J5.14 (Pin_14)
- net DISPLAY_D13: now also J5.2 (Pin_2); no longer J5.15 (Pin_15)
- net DISPLAY_D2: now also J5.13 (Pin_13); no longer J5.4 (Pin_4)
- net DISPLAY_D3: now also J5.12 (Pin_12); no longer J5.5 (Pin_5)
- net DISPLAY_D4: now also J5.11 (Pin_11); no longer J5.6 (Pin_6)
- net DISPLAY_D5: now also J5.10 (Pin_10); no longer J5.7 (Pin_7)
- net DISPLAY_D6: now also J5.9 (Pin_9); no longer J5.8 (Pin_8)
- net DISPLAY_D7: now also J5.8 (Pin_8); no longer J5.9 (Pin_9)
- net DISPLAY_D8: now also J5.7 (Pin_7); no longer J5.10 (Pin_10)
- net DISPLAY_D9: now also J5.6 (Pin_6); no longer J5.11 (Pin_11)
- net GND: now also J5.1 (Pin_1); no longer J5.16 (Pin_16)
- net PA18: now also R24.2; no longer U9.4 (TXD)
- net PA19: now also R25.2; no longer U9.5 (RXD)
- net SF_D+: now also U8.10 (DP1); no longer U8.8 (DP2)
- net SF_D-: now also U8.9 (DM1); no longer U8.7 (DM2)
- net UART_D+: now also U8.6 (DP3); no longer U8.10 (DP1)
- net UART_D-: now also U8.5 (DM3); no longer U8.9 (DM1)
- net I2C_SCL renamed PA26
- net I2C_SDA renamed PA27
- new net: R24.1, U9.4 (TXD)
- new net: R25.1, U9.5 (RXD)
- no-connect marks 14 -> 12

Commit message: update:
Parts:
- removed R3: 0R, Resistor_SMD:R_0402_1005Metric, symbol Device:R
- added C60, C61: TBD, Capacitor_SMD:C_0402_1005Metric, symbol Device:C
- added C62: 0.1u, Capacitor_SMD:C_0402_1005Metric, symbol Device:C
- added SW2: SW_SPDT, symbol Switch:SW_SPDT
- added U12: FM8625H, Package_LGA:Infineon_PG-TSNP-6-10_0.7x1.1mm_0.7x1.1mm_P0.4mm, symbol RF_Switch:BGS12WN6E6327
- R2: value 0R -> TBD_R
Connections:
- net GND: now also C60.2, C61.2, C62.2, SW2.1 (A), U12.2 (GND)
- net VDD33_1: now also C62.1, SW2.3 (C), U12.4 (VDD)
- net at AE2.1 (A): now also R2.2, C61.1
- net at AE1.1 (A): now also C17.1, R1.2; no longer R2.1
- new net: U1.53 (ANT), U12.5 (RFIN)
- new net RF1: C16.1, R1.1, U12.3 (RF1)
- new net RF2: C60.1, R2.1, U12.1 (RF2)
- new net RF_CTRL: SW2.2 (B), U12.6 (CTRL)
Other:
- moved on the sheet: AE1, J5

Commit message: update:
Parts:
- removed SW2: SW_SPDT, symbol Switch:SW_SPDT
- added R3: 1k, Resistor_SMD:R_0402_1005Metric, symbol Device:R
- added SW2: SK-3293S, My Switch:SW-SMD_SK-3293S_mini_7P, symbol Switch:SW_SPDT_321
Connections:
- net GND: now also SW2.1 (C)
- net RF1: now also C60.1, R2.1; no longer C16.1, R1.1
- net RF2: now also C16.1, R1.1; no longer C60.1, R2.1
- net RF_CTRL: now also R3.2
- net VDD33_1: now also SW2.3 (A)
- new net: R3.1, SW2.2 (B)
Other:
- sheet Audio ports: added PA_EN; removed none
